Commit message: add urscript.srv

File: ur_description/urdf/ur3.urdf.xacro (robot description, xacro)
@@ -289,4 +289,11 @@
       <child link="${prefix}tool0"/>
     </joint>
+    <!-- Connect tool0_controller to base using floating joint -->
+    <link name="${prefix}tool0_controller"/>
+    <joint name="${prefix}base-tool0_controller_floating_joint" type="floating">
+      <origin xyz="0 0 0" rpy="0 0 0"/>
+      <parent link="${prefix}base"/>
+      <child link="${prefix}tool0_controller"/>
+    </joint>
   </xacro:macro>
 </robot>

Commit message: sensor moveit config

File: ur_description/urdf/ur3.urdf.xacro (robot description, xacro)
@@ -290,10 +290,10 @@
     </joint>
     <!-- Connect tool0_controller to base using floating joint -->
-    <link name="${prefix}tool0_controller"/>
+    <!--link name="${prefix}tool0_controller"/>
     <joint name="${prefix}base-tool0_controller_floating_joint" type="floating">
       <origin xyz="0 0 0" rpy="0 0 0"/>
       <parent link="${prefix}base"/>
       <child link="${prefix}tool0_controller"/>
-    </joint>
+    </joint-->
   </xacro:macro>
 </robot>
